Commit message: Removes control config from baybot_description

File: baybot_description/urdf/baybot.gazebo.xacro (robot description, xacro)
@@ -1,54 +1,96 @@
 <?xml version="1.0"?>
 <robot xmlns:xacro="http://www.ros.org/wiki/xacro" name="rosbots" >
+<gazebo reference="wheel_left_link">
+  <mu1>1.0</mu1>
+  <mu2>1.0</mu2>
+  <kp>1000000.0</kp>
+  <kd>100.0</kd>
+  <minDepth>0.001</minDepth>
+  <maxVel>1.0</maxVel>
+</gazebo>
+<gazebo reference="wheel_right_link">
+  <mu1>1.0</mu1>
+  <mu2>1.0</mu2>
+  <kp>1000000.0</kp>
+  <kd>100.0</kd>
+  <minDepth>0.001</minDepth>
+  <maxVel>1.0</maxVel>
+</gazebo>
+<gazebo reference="base_link">
+  <material>Gazebo/Blue</material>
+  <mu1>0.3</mu1>
+  <mu2>0.3</mu2>
+  <sensor type="contact" name="bumpers">
+    <always_on>1</always_on>
+    <update_rate>50.0</update_rate>
+    <visualize>true</visualize>
+    <contact>
+      <collision>base_footprint_collision_base_link</collision>
+    </contact>
+  </sensor>
+</gazebo>
+<gazebo>
+  <plugin name="gazebo_ros_imu_controller" filename="libgazebo_ros_imu.so">
+    <!-- <robotNamespace></robotNamespace> -->
+    <topicName>imu/data</topicName>
+    <serviceName>imu/service</serviceName>
+    <bodyName>base_link</bodyName>
+    <gaussianNoise>0</gaussianNoise>
+    <rpyOffsets>0 0 0</rpyOffsets>
+    <updateRate>30.0</updateRate>
+    <alwaysOn>true</alwaysOn>
+    <gaussianNoise>0</gaussianNoise>
+  </plugin>
+</gazebo>
 <gazebo reference="camera_link">
-    <sensor type="camera" name="camera1">
-      <update_rate>30.0</update_rate>
-      <camera name="head">
-        <horizontal_fov>1.04</horizontal_fov>
-        <image>
-          <width>320</width>
-          <height>240</height>
-          <format>R8G8B8</format>
-        </image>
-        <clip>
-          <near>0.1</near>
-          <far>50</far>
-        </clip>
-      </camera>
-      <plugin name="camera_controller" filename="libgazebo_ros_camera.so">
-        <alwaysOn>true</alwaysOn>
-        <updateRate>0</updateRate>
-        <cameraName>camera1</cameraName>
-        <imageTopicName>image_raw</imageTopicName>
-        <cameraInfoTopicName>camera_info</cameraInfoTopicName>
-        <frameName>camera</frameName>
-        <hackBaseline>0.07</hackBaseline>
-        <distortionK1>0.0</distortionK1>
-        <distortionK2>0.0</distortionK2>
-        <distortionK3>0.0</distortionK3>
-        <distortionT1>0.0</distortionT1>
-        <distortionT2>0.0</distortionT2>
-      </plugin>
-    </sensor>
-  </gazebo>
-  <gazebo>
-    <plugin name="differential_drive_controller" filename="libgazebo_ros_diff_drive.so">
-        <legacyMode>false</legacyMode>
-        <alwaysOn>true</alwaysOn>
-        <publishWheelTF>true</publishWheelTF>
-        <publishTf>1</publishTf>
-        <publishWheelJointState>true</publishWheelJointState>
-        <updateRate>100.0</updateRate>
-        <leftJoint>wheel_left_joint</leftJoint>
-        <rightJoint>wheel_right_joint</rightJoint>
-        <wheelSeparation>1.1</wheelSeparation>
-        <wheelDiameter>0.52</wheelDiameter>
-        <wheelAcceleration>1.0</wheelAcceleration>
-        <torque>20</torque>
-        <commandTopic>/part2_cmr/cmd_vel</commandTopic>
-        <odometryTopic>odom</odometryTopic>
-        <odometryFrame>odom</odometryFrame>
-        <robotBaseFrame>base_link</robotBaseFrame>
+  <sensor type="camera" name="camera1">
+    <update_rate>30.0</update_rate>
+    <camera name="head">
+      <horizontal_fov>1.04</horizontal_fov>
+      <image>
+        <width>320</width>
+        <height>240</height>
+        <format>R8G8B8</format>
+      </image>
+      <clip>
+        <near>0.1</near>
+        <far>50</far>
+      </clip>
+    </camera>
+    <plugin name="camera_controller" filename="libgazebo_ros_camera.so">
+      <alwaysOn>true</alwaysOn>
+      <updateRate>0</updateRate>
+      <cameraName>camera1</cameraName>
+      <imageTopicName>image_raw</imageTopicName>
+      <cameraInfoTopicName>camera_info</cameraInfoTopicName>
+      <frameName>camera</frameName>
+      <hackBaseline>0.07</hackBaseline>
+      <distortionK1>0.0</distortionK1>
+      <distortionK2>0.0</distortionK2>
+      <distortionK3>0.0</distortionK3>
+      <distortionT1>0.0</distortionT1>
+      <distortionT2>0.0</distortionT2>
     </plugin>
+  </sensor>
+</gazebo>
+<gazebo>
+  <plugin name="differential_drive_controller" filename="libgazebo_ros_diff_drive.so">
+    <legacyMode>false</legacyMode>
+    <alwaysOn>true</alwaysOn>
+    <publishWheelTF>true</publishWheelTF>
+    <publishTf>1</publishTf>
+    <publishWheelJointState>true</publishWheelJointState>
+    <updateRate>100.0</updateRate>
+    <leftJoint>wheel_left_joint</leftJoint>
+    <rightJoint>wheel_right_joint</rightJoint>
+    <wheelSeparation>1.1</wheelSeparation>
+    <wheelDiameter>0.52</wheelDiameter>
+    <wheelAcceleration>1.0</wheelAcceleration>
+    <torque>20</torque>
+    <commandTopic>/part2_cmr/cmd_vel</commandTopic>
+    <odometryTopic>odom</odometryTopic>
+    <odometryFrame>odom</odometryFrame>
+    <robotBaseFrame>base_link</robotBaseFrame>
+  </plugin>
 </gazebo>
 </robot>

File: baybot_description/urdf/baybot.xacro (robot description, xacro)
@@ -5,66 +5,4 @@
     <origin xyz="0.155 0 0.4" rpy="0 0 0" />
   </xacro:asus_camera>
-  <gazebo reference="wheel_left_link">
-    <mu1>1.0</mu1>
-    <mu2>1.0</mu2>
-    <kp>1000000.0</kp>
-    <kd>100.0</kd>
-    <minDepth>0.001</minDepth>
-    <maxVel>1.0</maxVel>
-  </gazebo>
-  <gazebo reference="wheel_right_link">
-    <mu1>1.0</mu1>
-    <mu2>1.0</mu2>
-    <kp>1000000.0</kp>
-    <kd>100.0</kd>
-    <minDepth>0.001</minDepth>
-    <maxVel>1.0</maxVel>
-  </gazebo>
-  <gazebo reference="base_link">
-    <material>Gazebo/Blue</material>
-    <mu1>0.3</mu1>
-    <mu2>0.3</mu2>
-    <sensor type="contact" name="bumpers">
-      <always_on>1</always_on>
-      <update_rate>50.0</update_rate>
-      <visualize>true</visualize>
-      <contact>
-        <collision>base_footprint_collision_base_link</collision>
-      </contact>
-    </sensor>
-  </gazebo>
-  <gazebo>
-    <plugin name="gazebo_ros_imu_controller" filename="libgazebo_ros_imu.so">
-      <!-- <robotNamespace></robotNamespace> -->
-      <topicName>imu/data</topicName>
-      <serviceName>imu/service</serviceName>
-      <bodyName>base_link</bodyName>
-      <gaussianNoise>0</gaussianNoise>
-      <rpyOffsets>0 0 0</rpyOffsets>
-      <updateRate>30.0</updateRate>
-      <alwaysOn>true</alwaysOn>
-      <gaussianNoise>0</gaussianNoise>
-    </plugin>
-  </gazebo>
-  <gazebo>
-    <plugin name="differential_drive_controller" filename="libgazebo_ros_diff_drive.so">
-      <legacyMode>false</legacyMode>
-      <alwaysOn>true</alwaysOn>
-      <publishWheelTF>true</publishWheelTF>
-      <publishTf>1</publishTf>
-      <publishWheelJointState>true</publishWheelJointState>
-      <updateRate>100.0</updateRate>
-      <leftJoint>wheel_left_joint</leftJoint>
-      <rightJoint>wheel_right_joint</rightJoint>
-      <wheelSeparation>0.2756</wheelSeparation>
-      <wheelDiameter>0.1</wheelDiameter>
-      <wheelAcceleration>1.0</wheelAcceleration>
-      <torque>20</torque>
-      <commandTopic>/part2_cmr/cmd_vel</commandTopic>
-      <odometryTopic>odom</odometryTopic>
-      <odometryFrame>odom</odometryFrame>
-      <robotBaseFrame>base_link</robotBaseFrame>
-    </plugin>
-  </gazebo>
   <link name="base_footprint"/>
   <joint name="base_joint" type="fixed">

Commit message: Breaks out gazebo and rviz launchers/config into separate packages

File: baybot_description/urdf/baybot.gazebo.xacro (robot description, xacro)
@@ -1,4 +1,9 @@
 <?xml version="1.0"?>
-<robot xmlns:xacro="http://www.ros.org/wiki/xacro" name="rosbots" >
+<robot xmlns:xacro="http://www.ros.org/wiki/xacro" name="baybot" >
+<gazebo>
+  <plugin name="gazebo_ros_control" filename="libgazebo_ros_control.so">
+    <robotNamespace>$(arg robot_namespace)</robotNamespace>
+  </plugin>
+</gazebo>
 <gazebo reference="wheel_left_link">
   <mu1>1.0</mu1>
@@ -9,4 +14,13 @@
   <maxVel>1.0</maxVel>
 </gazebo>
+<transmission name="l_wheel_trans" type="SimpleTransmission">
+  <type>transmission_interface/SimpleTransmission</type>
+  <actuator name="l_wheel_motor">
+    <mechanicalReduction>1</mechanicalReduction>
+  </actuator>
+  <joint name="wheel_left_joint">
+    <hardwareInterface>hardware_interface/VelocityJointInterface</hardwareInterface>
+  </joint>
+</transmission>
 <gazebo reference="wheel_right_link">
   <mu1>1.0</mu1>
@@ -17,4 +31,13 @@
   <maxVel>1.0</maxVel>
 </gazebo>
+<transmission name="r_wheel_trans" type="SimpleTransmission">
+  <type>transmission_interface/SimpleTransmission</type>
+  <actuator name="r_wheel_motor">
+    <mechanicalReduction>1</mechanicalReduction>
+  </actuator>
+  <joint name="wheel_right_joint">
+    <hardwareInterface>hardware_interface/VelocityJointInterface</hardwareInterface>
+  </joint>
+</transmission>
 <gazebo reference="base_link">
   <material>Gazebo/Blue</material>
@@ -74,23 +97,3 @@
   </sensor>
 </gazebo>
-<gazebo>
-  <plugin name="differential_drive_controller" filename="libgazebo_ros_diff_drive.so">
-    <legacyMode>false</legacyMode>
-    <alwaysOn>true</alwaysOn>
-    <publishWheelTF>true</publishWheelTF>
-    <publishTf>1</publishTf>
-    <publishWheelJointState>true</publishWheelJointState>
-    <updateRate>100.0</updateRate>
-    <leftJoint>wheel_left_joint</leftJoint>
-    <rightJoint>wheel_right_joint</rightJoint>
-    <wheelSeparation>1.1</wheelSeparation>
-    <wheelDiameter>0.52</wheelDiameter>
-    <wheelAcceleration>1.0</wheelAcceleration>
-    <torque>20</torque>
-    <commandTopic>/part2_cmr/cmd_vel</commandTopic>
-    <odometryTopic>odom</odometryTopic>
-    <odometryFrame>odom</odometryFrame>
-    <robotBaseFrame>base_link</robotBaseFrame>
-  </plugin>
-</gazebo>
 </robot>

File: baybot_description/urdf/baybot.urdf.xacro (robot description, xacro)
@@ -1,5 +1,6 @@
 <?xml version="1.0" encoding="utf-8"?>
 <robot name="baybot" xmlns:xacro="http://www.ros.org/wiki/xacro">
-  <xacro:include filename="$(find baybot_description)/urdf/xtion.xacro"/>
+  <xacro:include filename="$(find baybot_description)/urdf/xtion.urdf.xacro"/>
+  <xacro:include filename="$(find baybot_description)/urdf/baybot.gazebo.xacro"/>
   <xacro:asus_camera name="xtion" parent="base_link">
     <origin xyz="0.155 0 0.4" rpy="0 0 0" />
@@ -57,5 +58,5 @@
     <parent link="base_link"/>
     <child link="wheel_left_link"/>
-    <origin xyz="0.067 -0.1378 0.05" rpy="-1.57 0 0"/>
+    <origin xyz="0.067 0.1378 0.05" rpy="-1.57 0 0"/>
     <axis xyz="0 0 1"/>
   </joint>
@@ -82,5 +83,5 @@
     <parent link="base_link"/>
     <child link="wheel_right_link"/>
-    <origin xyz="0.067 0.1378 0.05" rpy="-1.57 0 0"/>
+    <origin xyz="0.067 -0.1378 0.05" rpy="-1.57 0 0"/>
     <axis xyz="0 0 1"/>
   </joint>
@@ -90,5 +91,5 @@
         <cylinder length="0.027" radius="0.05"/>
       </geometry>
-      <origin rpy="0.0 0 0" xyz="0 0 0.195"/>
+      <origin rpy="0 0 0" xyz="0 0 0.195"/>
     </collision>
     <visual name="visual">
@@ -96,9 +97,9 @@
         <cylinder length="0.027" radius="0.05"/>
       </geometry>
-      <origin rpy="0.0 0 0" xyz="0 0 0"/>
+      <origin rpy="0 0 0" xyz="0 0 0"/>
     </visual>
     <inertial>
       <mass value="0.4" />
-      <origin xyz="0 0.0 0.3" />
+      <origin xyz="0 0 0.3" />
       <inertia ixx="0.001" ixy="0.0" ixz="0.0" iyy="0.001" iyz="0.0" izz="0.001" />
     </inertial>

File: baybot_description/urdf/xtion.urdf.xacro (robot description, xacro)
@@ -1,4 +1,4 @@
 <?xml version="1.0"?>
-<robot xmlns:xacro="http://ros.org/wiki/xacro">
+<robot xmlns:xacro="http://www.ros.org/wiki/xacro">
   <xacro:property name="M_PI" value="3.1415926535897931" />
   <xacro:macro name="asus_camera_model" params="name parent *origin">

Commit message: Fix everything.

File: baybot_description/urdf/baybot.gazebo.xacro (robot description, xacro)
@@ -19,5 +19,5 @@
     <mechanicalReduction>1</mechanicalReduction>
   </actuator>
-  <joint name="wheel_left_joint">
+  <joint name="l_wheel_joint">
     <hardwareInterface>hardware_interface/VelocityJointInterface</hardwareInterface>
   </joint>

File: baybot_description/urdf/baybot.urdf.xacro (robot description, xacro)
@@ -55,5 +55,5 @@
     </inertial>
   </link>
-  <joint name="wheel_left_joint" type="continuous">
+  <joint name="l_wheel_joint" type="continuous">
     <parent link="base_link"/>
     <child link="wheel_left_link"/>

Commit message: Consistent wheel names

File: baybot_description/urdf/baybot.gazebo.xacro (robot description, xacro)
@@ -36,5 +36,5 @@
     <mechanicalReduction>1</mechanicalReduction>
   </actuator>
-  <joint name="wheel_right_joint">
+  <joint name="r_wheel_joint">
     <hardwareInterface>hardware_interface/VelocityJointInterface</hardwareInterface>
   </joint>

File: baybot_description/urdf/baybot.urdf.xacro (robot description, xacro)
@@ -80,5 +80,5 @@
     </inertial>
   </link>
-  <joint name="wheel_right_joint" type="continuous">
+  <joint name="r_wheel_joint" type="continuous">
     <parent link="base_link"/>
     <child link="wheel_right_link"/>
